File: SerialSniffer_kicad/SerialSniffer_kicad.kicad_sch (KiCad schematic)
At the start: 24 parts, among them J1 DE9_Plug_MountingHoles, J2 DE9_Receptacle_MountingHoles, J3 Conn_01x10, J4 Conn_01x02, J5 Conn_02x02_Odd_Even, J6 Conn_02x02_Odd_Even, J7 STM32F401, J8 Conn_02x02_Odd_Even, U1 74HC14

Commit message: Initial
Parts:
- R3, R5: value 1k -> 100k
Changed lines of the file:
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@@
 			)
 		)
-		(property "Value" "1k"
+		(property "Value" "100k"
 			(at 55.88 27.9399 0)
 			(effects
@@
 			)
 		)
-		(property "Value" "1k"
+		(property "Value" "100k"
 			(at 55.88 54.6099 0)
 			(effects
